File: INV_Board.kicad_sch (KiCad schematic)
At the start: 216 parts, among them J11 Conn_01x05_Male

Commit message: Checkpoint before deleting MCU ISense
Parts:
- removed C30, C35: (no value), symbol Device:C_Small
- removed D22: (no value), symbol Diode:BAT48JFILM
- removed FL?: Filter_EMI_CommonMode, symbol Device:Filter_EMI_CommonMode
- removed J2, J3, J4: (no value), symbol Connector:Conn_01x02_Male
- removed J7: (no value), symbol Connector:Conn_01x03_Male
- removed J8: (no value), symbol Connector:Conn_ARM_JTAG_SWD_10
- removed L3: L_15uH_3A, symbol Device:L_Small
- removed NT1, NT3: (no value), symbol Device:NetTie_2
- removed NT2: Net-Tie_2, NetTie:NetTie-2_SMD_Pad0.5mm, symbol Device:NetTie_2
- removed Q10, Q11, Q12, Q7, Q8, Q9: (no value), symbol Transistor_FET:IPT015N10N5
- removed R53, R54: (no value), symbol Device:R_Small
- removed R? (x2): R_5.76K, symbol Device:R_Small
- removed TP1, TP2, TP3: (no value), symbol Connector:TestPoint
- removed U8: (no value), symbol Regulator_Switching:TPS61041DDC
- added C29: C_100pF_16V, Capacitor_SMD:C_0603_1608Metric, symbol Device:C_Small
- added D12, D5, D6: D_TVS, symbol Device:D_TVS
- added R33: R_4k7, Resistor_SMD:R_0603_1608Metric, symbol Device:R_Small
- added R43: R_10.2K, Resistor_SMD:R_0603_1608Metric, symbol Device:R_Small
- added R44: R_1.96K, Resistor_SMD:R_0603_1608Metric, symbol Device:R_Small
- C1: renamed from C22; value (none) -> C_0.1uF_100V; footprint (none) -> Capacitor_SMD:C_0603_1608Metric; LCSC C14663 -> C28233; Mouser Part no. 710-885012206071 -> (none); MouserAlt 603-CC603KRX7R8BB104 -> (none)
- C10: renamed from C23; value (none) -> C_0.1uF_100V; footprint (none) -> Capacitor_SMD:C_0603_1608Metric; LCSC C14663 -> C28233; Mouser Part no. 710-885012206071 -> (none); MouserAlt 603-CC603KRX7R8BB104 -> (none)
- C11, C12, C14, C15: renamed from C?; LCSC (none) -> C53987
- C16: renamed from C29; value (none) -> C_100pF_16V; footprint (none) -> Capacitor_SMD:C_0603_1608Metric; Mouser Part no. 710-885012006023 -> (none); MouserAlt 603-CC603KRX7R7BB101 -> (none)
- C17: renamed from C?; footprint Capacitor_SMD:C_0805_2012Metric -> Capacitor_SMD:C_0603_1608Metric; Mouser Part no. 710-885012207128 -> (none); MouserAlt 581-08051C104M4Z2A -> (none)
- C18: renamed from C?; LCSC C72477 -> C72477
- C19: renamed from C41; value (none) -> C_100pF_16V; footprint (none) -> Capacitor_SMD:C_0603_1608Metric; Mouser Part no. 710-885012006023 -> (none); MouserAlt 603-CC603KRX7R7BB101 -> (none)
- C2, C3: renamed from C?; LSCS potential C650969 -> (none); Mouser Part no. 581-12101C475K4T2A -> (none); MouserAlt 963-HMK325C7475MM-PE -> (none)
- C20: renamed from C42; value (none) -> C_100pF_16V; footprint (none) -> Capacitor_SMD:C_0603_1608Metric; Mouser Part no. 710-885012006023 -> (none); MouserAlt 603-CC603KRX7R7BB101 -> (none)
- C21, C30: renamed from C?; footprint (none) -> Capacitor_SMD:C_0603_1608Metric; LCSC (none) -> C27920
- C22, C31: renamed from C?; footprint (none) -> Capacitor_SMD:C_0603_1608Metric; LCSC (none) -> C1634
- C24, C33: renamed from C?; footprint (none) -> Capacitor_SMD:C_0603_1608Metric; LCSC (none) -> C53987
- C25, C37, C5: renamed from C?; Mouser Part no. 963-TMK107B7105MA-T -> (none); MouserAlt 963-TMK107B7105KA-T -> (none)
- C34: renamed from C8; value (none) -> C_1uF_100V; footprint (none) -> Capacitor_SMD:C_0603_1608Metric; LCSC C15849 -> C91151; Mouser Part no. 963-TMK107B7105MA-T -> (none); MouserAlt 963-TMK107B7105KA-T -> (none)
- C35: renamed from C3; value (none) -> C_1uF_100V; footprint (none) -> Capacitor_SMD:C_0603_1608Metric; LCSC C15849 -> C91151; Mouser Part no. 963-TMK107B7105MA-T -> (none); MouserAlt 963-TMK107B7105KA-T -> (none)
- C36: renamed from C7; value (none) -> C_1uF_100V; footprint (none) -> Capacitor_SMD:C_0603_1608Metric; LCSC C15849 -> C91151; Mouser Part no. 963-TMK107B7105MA-T -> (none); MouserAlt 963-TMK107B7105KA-T -> (none)
- C38: renamed from C10; value (none) -> C_1uF_100V; footprint (none) -> Capacitor_SMD:C_0603_1608Metric; LCSC C15849 -> C91151; Mouser Part no. 963-TMK107B7105MA-T -> (none); MouserAlt 963-TMK107B7105KA-T -> (none)
- C39: renamed from C4; value (none) -> C_1uF_100V; footprint (none) -> Capacitor_SMD:C_0603_1608Metric; LCSC C15849 -> C91151; Mouser Part no. 963-TMK107B7105MA-T -> (none); MouserAlt 963-TMK107B7105KA-T -> (none)
- C4: renamed from C15; value (none) -> C_0.1uF_100V; footprint (none) -> Capacitor_SMD:C_0603_1608Metric; Mouser Part no. 710-885012207128 -> (none); MouserAlt 581-08051C104M4Z2A -> (none)
- C40: renamed from C9; value (none) -> C_1uF_100V; footprint (none) -> Capacitor_SMD:C_0603_1608Metric; LCSC C15849 -> C91151; Mouser Part no. 963-TMK107B7105MA-T -> (none); MouserAlt 963-TMK107B7105KA-T -> (none)
- C41: renamed from C27; Mouser Part no. 647-UVZ2A471MHD -> (none); MouserAlt 661-EKY10ELL681ML40S -> (none)
- C42: renamed from C28; value (none) -> CP_470uF+; footprint (none) -> Capacitor_THT:CP_Radial_D16.0mm_P7.50mm; Mouser Part no. 647-UVZ2A471MHD -> (none); MouserAlt 661-EKY10ELL681ML40S -> (none)
- C46: renamed from C59; value (none) -> CP_470uF+; footprint (none) -> Capacitor_THT:CP_Radial_D16.0mm_P7.50mm; Mouser Part no. 647-UVZ2A471MHD -> (none); MouserAlt 661-EKY10ELL681ML40S -> (none)
- C47: renamed from C33; value (none) -> C_1uF_100V; footprint (none) -> Capacitor_SMD:C_0603_1608Metric; LCSC C13832 -> C91151; LSCS potential C13832 -> (none); Mouser Part no. 581-12101C475K4T2A -> (none); MouserAlt 963-HMK325C7475MM-PE -> (none)
- C48: renamed from C12; value (none) -> C_1uF_100V; footprint (none) -> Capacitor_SMD:C_0603_1608Metric; LCSC C13832 -> C91151; LSCS potential C13832 -> (none); Mouser Part no. 581-12101C475K4T2A -> (none); MouserAlt 963-HMK325C7475MM-PE -> (none)
- C49: renamed from C11; value (none) -> CP_470uF+; footprint (none) -> Capacitor_THT:CP_Radial_D16.0mm_P7.50mm; Mouser Part no. 647-UVZ2A471MHD -> (none); MouserAlt 661-EKY10ELL681ML40S -> (none)
- C50: renamed from C51; value (none) -> C_1uF_100V; footprint (none) -> Capacitor_SMD:C_0603_1608Metric; LCSC C13832 -> C91151; Mouser Part no. 710-885012207128 -> (none); MouserAlt 581-08051C104M4Z2A -> (none)
- C51: renamed from C52; value (none) -> C_1uF_100V; footprint (none) -> Capacitor_SMD:C_0603_1608Metric; LCSC C13832 -> C91151; Mouser Part no. 710-885012207128 -> (none); MouserAlt 581-08051C104M4Z2A -> (none)
- C52: renamed from C13; value (none) -> C_0.1uF_100V; footprint (none) -> Capacitor_SMD:C_0603_1608Metric; Mouser Part no. 710-885012207128 -> (none); MouserAlt 581-08051C104M4Z2A -> (none)
- C53: value (none) -> C_1uF_100V; footprint (none) -> Capacitor_SMD:C_0603_1608Metric; LCSC C13832 -> C91151; Mouser Part no. 710-885012207128 -> (none); MouserAlt 581-08051C104M4Z2A -> (none)
- C54: renamed from C37; value (none) -> C_1uF_100V; footprint (none) -> Capacitor_SMD:C_0603_1608Metric; LCSC C13832 -> C91151; LSCS potential C13832 -> (none); Mouser Part no. 581-12101C475K4T2A -> (none); MouserAlt 963-HMK325C7475MM-PE -> (none)
- C55: renamed from C1; value (none) -> C_1uF_100V; footprint (none) -> Capacitor_SMD:C_0603_1608Metric; LCSC C13832 -> C91151; LSCS potential C13832 -> (none); Mouser Part no. 581-12101C475K4T2A -> (none); MouserAlt 963-HMK325C7475MM-PE -> (none)
- C56: renamed from C54; value (none) -> C_1uF_100V; footprint (none) -> Capacitor_SMD:C_0603_1608Metric; LCSC C13832 -> C91151; Mouser Part no. 710-885012207128 -> (none); MouserAlt 581-08051C104M4Z2A -> (none)
- C57: renamed from C32; value (none) -> C_1uF_100V; footprint (none) -> Capacitor_SMD:C_0603_1608Metric; LCSC C13832 -> C91151; LSCS potential C13832 -> (none); Mouser Part no. 581-12101C475K4T2A -> (none); MouserAlt 963-HMK325C7475MM-PE -> (none)
- C58: renamed from C55; value (none) -> C_1uF_100V; footprint (none) -> Capacitor_SMD:C_0603_1608Metric; LCSC C13832 -> C91151; Mouser Part no. 710-885012207128 -> (none); MouserAlt 581-08051C104M4Z2A -> (none)
- C59: renamed from C31; value (none) -> C_1uF_100V; footprint (none) -> Capacitor_SMD:C_0603_1608Metric; LCSC C13832 -> C91151; LSCS potential C13832 -> (none); Mouser Part no. 581-12101C475K4T2A -> (none); MouserAlt 963-HMK325C7475MM-PE -> (none)
- C6: renamed from C2; value (none) -> C_1uF_100V; footprint (none) -> Capacitor_SMD:C_0603_1608Metric; LCSC C15849 -> C91151; Mouser Part no. 963-TMK107B7105MA-T -> (none); MouserAlt 963-TMK107B7105KA-T -> (none)
- C60: renamed from C5; value (none) -> C_1uF_100V; footprint (none) -> Capacitor_SMD:C_0603_1608Metric; LCSC C28233 -> C91151; Mouser Part no. 710-885012207128 -> (none); MouserAlt 581-08051C104M4Z2A -> (none)
- C61: renamed from C56; value (none) -> C_1uF_100V; footprint (none) -> Capacitor_SMD:C_0603_1608Metric; LCSC C13832 -> C91151; Mouser Part no. 710-885012207128 -> (none); MouserAlt 581-08051C104M4Z2A -> (none)
- C62: renamed from C44; value (none) -> C_1uF_100V; footprint (none) -> Capacitor_SMD:C_0603_1608Metric; LCSC C13832 -> C91151; Mouser Part no. 710-885012207128 -> (none); MouserAlt 581-08051C104M4Z2A -> (none)
- C63: renamed from C26; value (none) -> C_0.1uF_100V; footprint (none) -> Capacitor_SMD:C_0603_1608Metric; LCSC C14858 -> C28233; Mouser Part no. 710-885012006023 -> (none); MouserAlt 603-CC603KRX7R7BB101 -> (none)
- C64: renamed from C57; value (none) -> C_1uF_100V; footprint (none) -> Capacitor_SMD:C_0603_1608Metric; LCSC C13832 -> C91151; Mouser Part no. 710-885012207128 -> (none); MouserAlt 581-08051C104M4Z2A -> (none)
- C65: renamed from C24; value (none) -> C_0.1uF_100V; footprint (none) -> Capacitor_SMD:C_0603_1608Metric; LCSC C14858 -> C28233; Mouser Part no. 710-885012006023 -> (none); MouserAlt 603-CC603KRX7R7BB101 -> (none)
- C66: renamed from C25; value (none) -> C_0.1uF_100V; footprint (none) -> Capacitor_SMD:C_0603_1608Metric; LCSC C14858 -> C28233; Mouser Part no. 710-885012006023 -> (none); MouserAlt 603-CC603KRX7R7BB101 -> (none)
- C67: renamed from C45; value (none) -> C_1uF_100V; footprint (none) -> Capacitor_SMD:C_0603_1608Metric; LCSC C13832 -> C91151; Mouser Part no. 710-885012207128 -> (none); MouserAlt 581-08051C104M4Z2A -> (none)
- C68: renamed from C14; value (none) -> C_0.1uF_100V; footprint (none) -> Capacitor_SMD:C_0603_1608Metric; Mouser Part no. 710-885012207128 -> (none); MouserAlt 581-08051C104M4Z2A -> (none)
- C69: renamed from C46; value (none) -> C_1uF_100V; footprint (none) -> Capacitor_SMD:C_0603_1608Metric; LCSC C13832 -> C91151; Mouser Part no. 710-885012207128 -> (none); MouserAlt 581-08051C104M4Z2A -> (none)
- C7: renamed from C39; value (none) -> C_0.1uF_100V; footprint (none) -> Capacitor_SMD:C_0603_1608Metric; LCSC C14663 -> C28233; Mouser Part no. 710-885012206071 -> (none); MouserAlt 603-CC603KRX7R8BB104 -> (none)
- C70: renamed from C47; value (none) -> C_1uF_100V; footprint (none) -> Capacitor_SMD:C_0603_1608Metric; LCSC C13832 -> C91151; Mouser Part no. 710-885012207128 -> (none); MouserAlt 581-08051C104M4Z2A -> (none)
- C71: renamed from C21; value (none) -> C_0.1uF_100V; footprint (none) -> Capacitor_SMD:C_0603_1608Metric; LCSC C14858 -> C28233; Mouser Part no. 710-885012006023 -> (none); MouserAlt 603-CC603KRX7R7BB101 -> (none)
- C72: renamed from C48; value (none) -> C_1uF_100V; footprint (none) -> Capacitor_SMD:C_0603_1608Metric; LCSC C13832 -> C91151; Mouser Part no. 710-885012207128 -> (none); MouserAlt 581-08051C104M4Z2A -> (none)
- C73: renamed from C49; value (none) -> C_1uF_100V; footprint (none) -> Capacitor_SMD:C_0603_1608Metric; LCSC C13832 -> C91151; Mouser Part no. 710-885012207128 -> (none); MouserAlt 581-08051C104M4Z2A -> (none)
- C74: renamed from C50; value (none) -> C_1uF_100V; footprint (none) -> Capacitor_SMD:C_0603_1608Metric; LCSC C13832 -> C91151; Mouser Part no. 710-885012207128 -> (none); MouserAlt 581-08051C104M4Z2A -> (none)
- C8: renamed from C16; Mouser Part no. 963-TMK107B7105MA-T -> (none); MouserAlt 963-TMK107B7105KA-T -> (none)
- C9: renamed from C6; value (none) -> C_0.1uF_100V; footprint (none) -> Capacitor_SMD:C_0603_1608Metric; LCSC C14663 -> C28233; Mouser Part no. 710-885012206071 -> (none); MouserAlt 603-CC603KRX7R8BB104 -> (none)
- D1, D2: renamed from D?; footprint Diode_SMD:D_0603_1608Metric -> (none)
- D10: renamed from D18; value (none) -> D_TVS; Mouser Part no. DNP -> (none)
- D11: renamed from D5; footprint (none) -> Diode_SMD:D_MiniMELF; Mouser Part no. 863-MM3Z3V3ST1G -> (none); MouserAlt 863-MM3Z3V3T1G -> (none)
- D13: renamed from D6; footprint (none) -> Diode_SMD:D_MiniMELF; Mouser Part no. 863-MM3Z3V3ST1G -> (none); MouserAlt 863-MM3Z3V3T1G -> (none)
- D14, D4, D8: renamed from D?; footprint (none) -> Diode_SMD:D_SOD-123F
- D15: renamed from D3; value (none) -> D_Sch_100V_2A; footprint (none) -> Diode_SMD:D_SOD-123F; Mouser Part no. 863-MBR2H200SFT1G -> (none); MouserAlt 821-SS215LWRVG -> (none)
- D16: renamed from D1; value (none) -> D_Sch_100V_2A; footprint (none) -> Diode_SMD:D_SOD-123F; Mouser Part no. 863-MBR2H200SFT1G -> (none); MouserAlt 821-SS215LWRVG -> (none)
- D17: renamed from D2; value (none) -> D_Sch_100V_2A; footprint (none) -> Diode_SMD:D_SOD-123F; Mouser Part no. 863-MBR2H200SFT1G -> (none); MouserAlt 821-SS215LWRVG -> (none)
- D18: renamed from D15; value (none) -> D_TVS; Mouser Part no. 576-SMCJ54CA -> (none); MouserAlt 652-SMCJ54CA -> (none)
- D19: renamed from D7; value (none) -> D_Zener_3V3; footprint (none) -> Diode_SMD:D_MiniMELF; LCSC C145245 -> C8056; Mouser Part no. 863-MM3Z3V3ST1G -> (none); MouserAlt 863-MM3Z3V3T1G -> (none)
- D20: renamed from D13; value (none) -> D_Zener_16V; footprint (none) -> Diode_SMD:D_SOD-123; LCSC C150089 -> C27754; Mouser Part no. 863-MM3Z16VST1G -> (none); MouserAlt 621-DDZ16CSF-7 -> (none)
- D21: renamed from D14; value (none) -> D_Zener_16V; footprint (none) -> Diode_SMD:D_SOD-123; LCSC C150089 -> C27754; Mouser Part no. 863-MM3Z16VST1G -> (none); MouserAlt 621-DDZ16CSF-7 -> (none)
- D22: renamed from D9; value (none) -> D_Zener_16V; footprint (none) -> Diode_SMD:D_SOD-123; LCSC C150089 -> C27754; Mouser Part no. 863-MM3Z16VST1G -> (none); MouserAlt 621-DDZ16CSF-7 -> (none)
- D23: renamed from D10; value (none) -> D_Zener_16V; footprint (none) -> Diode_SMD:D_SOD-123; LCSC C150089 -> C27754; Mouser Part no. 863-MM3Z16VST1G -> (none); MouserAlt 621-DDZ16CSF-7 -> (none)
- D24: renamed from D11; value (none) -> D_Zener_16V; footprint (none) -> Diode_SMD:D_SOD-123; LCSC C150089 -> C27754; Mouser Part no. 863-MM3Z16VST1G -> (none); MouserAlt 621-DDZ16CSF-7 -> (none)
- D25: renamed from D12; value (none) -> D_Zener_16V; footprint (none) -> Diode_SMD:D_SOD-123; LCSC C150089 -> C27754; Mouser Part no. 863-MM3Z16VST1G -> (none); MouserAlt 621-DDZ16CSF-7 -> (none)
- D26: renamed from D8; value (none) -> D_Zener_3V3; footprint (none) -> Diode_SMD:D_MiniMELF; LCSC C145245 -> C8056; Mouser Part no. 863-MM3Z3V3ST1G -> (none); MouserAlt 863-MM3Z3V3T1G -> (none)
- D3: renamed from D?; Mouser Part no. 710-150060AS75000 -> (none); MouserAlt 710-150060VS75000 -> (none)
- D7: renamed from D17; value (none) -> D_TVS; Mouser Part no. DNP -> (none)
- D9: renamed from D23; footprint (none) -> Diode_SMD:D_MiniMELF; Mouser Part no. 863-MM3Z3V3ST1G -> (none); MouserAlt 863-MM3Z3V3T1G -> (none)
- J3: renamed from J9; footprint (none) -> Connector_PinHeader_2.54mm:PinHeader_1x06_P2.54mm_Vertical
- J4: renamed from J12; footprint (none) -> Connector_JST:JST_PH_B6B-PH-K_1x06_P2.00mm_Vertical; RS No. B6B-PH-K-S(LF)(SN) -> (none)
- J5: renamed from J6; footprint (none) -> Connector_JST:JST_PH_B8B-PH-K_1x08_P2.00mm_Vertical
- J7: renamed from J11; footprint Connector_Molex:Molex_PicoBlade_53047-0510_1x05_P1.25mm_Vertical -> Connector_JST:JST_PH_B5B-PH-K_1x05_P2.00mm_Vertical
- J8: renamed from J10; footprint (none) -> INV_Board:XT60
- L1: footprint Inductor_SMD:L_Bourns-SRN8040_8x8.15mm -> Inductor_SMD:L_Bourns_SRP7028A_7.3x6.6mm; LSCS potential C149588 -> (none)
- L2, L3: renamed from L?; footprint (none) -> Inductor_SMD:L_Bourns_SRP7028A_7.3x6.6mm; LSCS potential C182182 -> (none)
- Q1: renamed from Q?; LCSC (none) -> C8545
- Q2: renamed from Q?; LCSC (none) -> C15127
- Q3: renamed from Q5; value (none) -> CRSS037N10N; footprint (none) -> Package_TO_SOT_SMD:TO-263-2
- Q4: renamed from Q6; value (none) -> CRSS037N10N; footprint (none) -> Package_TO_SOT_SMD:TO-263-2
- Q5: renamed from Q1; value (none) -> CRSS037N10N; footprint (none) -> Package_TO_SOT_SMD:TO-263-2
- Q6: renamed from Q2; value (none) -> CRSS037N10N; footprint (none) -> Package_TO_SOT_SMD:TO-263-2
- Q7: renamed from Q3; value (none) -> CRSS037N10N; footprint (none) -> Package_TO_SOT_SMD:TO-263-2
- Q8: renamed from Q4; value (none) -> CRSS037N10N; footprint (none) -> Package_TO_SOT_SMD:TO-263-2
- R10: renamed from R41; value (none) -> R_1.5k; footprint (none) -> Resistor_SMD:R_0603_1608Metric
- R11: renamed from R35; footprint (none) -> Resistor_SMD:R_0603_1608Metric
- R12: renamed from R42; value (none) -> R_1.5k; footprint (none) -> Resistor_SMD:R_0603_1608Metric
- R13: renamed from R47; value (none) -> R_100; footprint (none) -> Resistor_SMD:R_0603_1608Metric
- R14: renamed from R48; value (none) -> R_100; footprint (none) -> Resistor_SMD:R_0603_1608Metric
- R15: renamed from R46; footprint (none) -> Resistor_SMD:R_0603_1608Metric
- R16, R35: renamed from R?; footprint (none) -> Resistor_SMD:R_0603_1608Metric; LCSC (none) -> C23189
- R17: renamed from R58; value (none) -> R_30K; footprint (none) -> Resistor_SMD:R_0603_1608Metric
- R18: renamed from R59; value (none) -> R_30K; footprint (none) -> Resistor_SMD:R_0603_1608Metric
- R19: renamed from R64; footprint (none) -> Resistor_SMD:R_0603_1608Metric
- R20: renamed from R55; value (none) -> R_1.5k; footprint (none) -> Resistor_SMD:R_0603_1608Metric
- R21: renamed from R38; value (none) -> R_1.5k; footprint (none) -> Resistor_SMD:R_0603_1608Metric
- R22: renamed from R57; value (none) -> R_1.5k; footprint (none) -> Resistor_SMD:R_0603_1608Metric
- R23: renamed from R60; value (none) -> R_30K; footprint (none) -> Resistor_SMD:R_0603_1608Metric
- R24: renamed from R61; value (none) -> R_30K; footprint (none) -> Resistor_SMD:R_0603_1608Metric
- R25: renamed from R39; value (none) -> R_1.5k; footprint (none) -> Resistor_SMD:R_0603_1608Metric
- R26: renamed from R65; footprint (none) -> Resistor_SMD:R_0603_1608Metric
- R27: renamed from R37; value (none) -> R_1.5k; footprint (none) -> Resistor_SMD:R_0603_1608Metric
- R28: renamed from R?; value R_5.76K -> R_10.2K; footprint (none) -> Resistor_SMD:R_0603_1608Metric; LCSC (none) -> C25804
- R29: renamed from R?; value R_5.76K -> R_3.24K; footprint (none) -> Resistor_SMD:R_0603_1608Metric; LCSC (none) -> C22978
- R3: renamed from R19; value (none) -> R_590K; footprint (none) -> Resistor_SMD:R_0603_1608Metric; LCSC C22809 -> C23203
- R30: renamed from R56; footprint (none) -> Resistor_SMD:R_0603_1608Metric
- R31: renamed from R62; value (none) -> R_30K; footprint (none) -> Resistor_SMD:R_0603_1608Metric
- R32: renamed from R63; value (none) -> R_30K; footprint (none) -> Resistor_SMD:R_0603_1608Metric
- R34: renamed from R66; footprint (none) -> Resistor_SMD:R_0603_1608Metric
- R36: renamed from R28; value (none) -> R_1.5k; footprint (none) -> Resistor_SMD:R_0603_1608Metric
- R37: renamed from R29; footprint (none) -> Resistor_SMD:R_0603_1608Metric
- R38: renamed from R8; footprint (none) -> Resistor_SMD:R_0603_1608Metric
- R39: renamed from R2; footprint (none) -> Resistor_SMD:R_0603_1608Metric
- R4: renamed from R20; footprint (none) -> Resistor_SMD:R_0603_1608Metric
- R40: renamed from R7; footprint (none) -> Resistor_SMD:R_0603_1608Metric
- R41: renamed from R30; value (none) -> R_1.5k; footprint (none) -> Resistor_SMD:R_0603_1608Metric
- R42: renamed from R31; footprint (none) -> Resistor_SMD:R_0603_1608Metric
- R45: renamed from R11; footprint (none) -> Resistor_SMD:R_0603_1608Metric
- R46: renamed from R9; footprint (none) -> Resistor_SMD:R_0603_1608Metric
- R47: renamed from R12; footprint (none) -> Resistor_SMD:R_0603_1608Metric
- R48: renamed from R6; footprint (none) -> Resistor_SMD:R_0603_1608Metric
- R49: renamed from R3; footprint (none) -> Resistor_SMD:R_0603_1608Metric
- R5: renamed from R40; value (none) -> R_1.5k; footprint (none) -> Resistor_SMD:R_0603_1608Metric
- R50: renamed from R10; footprint (none) -> Resistor_SMD:R_0603_1608Metric
- R51: renamed from R32; value (none) -> R_1.5k; footprint (none) -> Resistor_SMD:R_0603_1608Metric
- R52: renamed from R27; value (none) -> Shunt; footprint (none) -> Resistor_SMD:R_2512_6332Metric
- R53: renamed from R25; value (none) -> Shunt; footprint (none) -> Resistor_SMD:R_2512_6332Metric
- R54: renamed from R26; value (none) -> Shunt; footprint (none) -> Resistor_SMD:R_2512_6332Metric
- R55: renamed from R14; value (none) -> Shunt; footprint (none) -> Resistor_SMD:R_2512_6332Metric
- R56: renamed from R1; value (none) -> Shunt; footprint (none) -> Resistor_SMD:R_2512_6332Metric
- R57: renamed from R13; value (none) -> Shunt; footprint (none) -> Resistor_SMD:R_2512_6332Metric
- R58: renamed from R33; footprint (none) -> Resistor_SMD:R_0603_1608Metric
- R59: renamed from R17; footprint (none) -> Resistor_SMD:R_0603_1608Metric
- R60: renamed from R18; footprint (none) -> Resistor_SMD:R_0603_1608Metric
- R61: renamed from R4; footprint (none) -> Resistor_SMD:R_0603_1608Metric
- R62: renamed from R5; footprint (none) -> Resistor_SMD:R_0603_1608Metric
- R63: renamed from R15; footprint (none) -> Resistor_SMD:R_0603_1608Metric
- R64: renamed from R16; footprint (none) -> Resistor_SMD:R_0603_1608Metric
- R65: renamed from R24; footprint (none) -> Resistor_SMD:R_0603_1608Metric
- R66: renamed from R23; value (none) -> R_1.5k; footprint (none) -> Resistor_SMD:R_0603_1608Metric
- R7: renamed from R34; footprint (none) -> Resistor_SMD:R_0603_1608Metric
- R8, R9: renamed from R?; value R_5.76K -> R_60; footprint (none) -> Resistor_SMD:R_0603_1608Metric; LCSC (none) -> C23220
- TH1: footprint (none) -> Resistor_SMD:R_0603_1608Metric
- U1: renamed from U2; footprint (none) -> Package_QFP:LQFP-48_7x7mm_P0.5mm
- U10: renamed from U3; footprint (none) -> Package_SO:SOIC-8_3.9x4.9mm_P1.27mm
- U11: renamed from U4; footprint (none) -> Package_SO:SOIC-8_3.9x4.9mm_P1.27mm
- U4: renamed from U1; footprint (none) -> Package_TO_SOT_SMD:SOT-23-6; LCSC (none) -> C2058943
- U5, U8: renamed from U?; footprint (none) -> Package_SO:SOIC-8-1EP_3.9x4.9mm_P1.27mm_EP2.29x3mm_ThermalVias; LCSC C9865 -> C9865
- U6: renamed from U9; footprint (none) -> Package_TO_SOT_SMD:SOT-23-6; LCSC (none) -> C2058943
- U7: renamed from U10; footprint (none) -> Package_TO_SOT_SMD:SOT-23-6; LCSC (none) -> C2058943
- U9: renamed from U5; footprint (none) -> Package_SO:SOIC-8_3.9x4.9mm_P1.27mm
- gave numbers to parts that had none: 14
- renumbered C17 to C13
Connections:
- net SGU is gone; now on net GND: U4.4 (-)
- net SGV is gone; now on net GND: U6.4 (-)
- net SGW is gone; now on net GND: U7.4 (-)
- net +12V: now also C23.1, C32.1, U5.2 (VIN), U8.2 (VIN); no longer C23.2, C32.2
- net +3V3: now also R33.1
- net +5V: now also R43.1
- net GND: now also C21.2, C22.2, C23.2, C24.2, C26.1, C27.1, C28.1, C30.2, C31.2, C32.2, C33.2, C43.1, C44.1, C45.1, D14.2 (A), D8.2 (A), R29.2, U5.7 (GND), U8.7 (GND), C29.2, D12.2 (A2), D5.2 (A2), D6.2 (A2), R44.2
- net ISU_MCU: no longer U1.11 (PA1)
- net ISV_MCU: no longer U1.17 (PA7)
- net ISW_MCU: no longer U1.18 (PB0)
- net STRx: now also D5.1 (A1)
- net STTx: now also D6.1 (A1)
- net Motor_T: now reaches J4.5 (Pin_5)
- net Motor_T: now also C29.1, D12.1 (A1), R33.2
- net at C12.2, J6.4 (Pin_4), R9.2: now also D2.2 (A2), U2.6 (CANL)
- net at D1.2 (A2), U2.7 (CANH): now also C11.2, J6.1 (Pin_1), R8.1
- net at U8.5 (VSENSE): now also R43.2, R44.1
Other:
- moved on the sheet: C16, C19, C20, C21, C22, C23, C24, C25, C26, C27, C28, C30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
