File: INV_Board.kicad_sch (KiCad schematic)
At the start: 181 parts, among them J6 Conn_01x08_Female, J7 Conn_01x05_Male, Q1 2N7002, Q2 AO3401A, Q3 CRSS037N10N, Q4 CRSS037N10N, Q5 CRSS037N10N, Q6 CRSS037N10N, Q7 CRSS037N10N, Q8 CRSS037N10N, U12 SMF05CT1G, U13 SMF05CT1G, U14 SMF05CT1G, U2 TJA1051T, U3 MP9486A, U5 TPS54331DR, U8 TPS54331DR, X1 ASE-xxxMHz

Commit message: Update progress
Parts:
- removed C14, C15: C_4.7nF, Capacitor_SMD:C_0603_1608Metric, symbol Device:C_Small
- removed R8, R9: R_60, Resistor_SMD:R_0603_1608Metric, symbol Device:R_Small
Connections:
- net I2CSCL: no longer J5.7 (Pin_7), R21.2, U1.46 (PB9), U14.3 (K)
- net Motor_T: now also U12.3 (K); no longer U12.6 (K)
- net at J4.2 (Pin_2), R12.2, R15.2: now also U12.6 (K); no longer U12.3 (K)
- net at C12.2, J6.4 (Pin_4), U13.3 (K)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: now also J6.3 (Pin_3)
- net at C11.2, J6.1 (Pin_1), U13.1 (K)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: now also J6.2 (Pin_2)
- new net I2CSDA: J5.7 (Pin_7), R21.2, U1.46 (PB9), U14.3 (K)

Commit message: 00A revision as ordered
00A version of board has been ordered for assembly. Warning: this commit contains some fixes which were not part of the order
Parts:
- C13, C23, C26, C27, C28, C32, C43, C44, C45: LCSC C96446 -> C96446
- C34, C35, C36, C38, C39, C40, C47, C48, C50, C51, C53, C54, C55, C56, C57, C58, C59, C6, C60, C61, C62, C64, C67, C69, C70, C72, C73, C74: footprint Capacitor_SMD:C_0603_1608Metric -> Capacitor_SMD:C_0805_2012Metric
- D11, D13, D9: value (none) -> D_Zener_3v3
- D20, D21, D22, D23, D24, D25: LCSC C27754 -> C27754
- J3: value (none) -> Conn_01x06_Male
- J4: value (none) -> Conn_01x06_Female
- J5: value (none) -> Conn_01x08_Female
- J8: value (none) -> Conn_01x02_Male
- Q2: LCSC C15127 -> C15127
- R11, R15, R30, R4, R7: value (none) -> R_4k7
- R19, R26, R34: value (none) -> R_150
- R37, R42, R58, R65: value (none) -> R_82k
- R38, R39, R40, R45, R46, R47, R48, R49, R50: value (none) -> R_5
- TH1: value (none) -> Thermistor_NTC
- U1: value (none) -> STM32F303CBTx
- U10, U11, U9: value (none) -> IR2181
- U12, U13, U14: LCSC (none) -> C15879
- U2: LCSC (none) -> C6952
- U4, U6, U7: value (none) -> INA181
- U5, U8: LCSC C9865 -> C9865
Other:
- title: MESC_FOC_ESC -> SQESC_FOC_ESC
- moved on the sheet: C11, C12, C34, C36, C38, C40, C47, C48, C5, C52, C54, C59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
