File: _autosave-INV_Board.kicad_sch (KiCad schematic)
At the start: 181 parts, among them J6 Conn_01x08_Female, J7 Conn_01x05_Male, Q1 2N7002, Q2 AO3401A, Q3 CRSS037N10N, Q4 CRSS037N10N, Q5 CRSS037N10N, Q6 CRSS037N10N, Q7 CRSS037N10N, Q8 CRSS037N10N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

Commit message: Save progress
Parts:
- removed C14, C15: C_4.7nF, Capacitor_SMD:C_0603_1608Metric, symbol Device:C_Small
- removed R8, R9: R_60, Resistor_SMD:R_0603_1608Metric, symbol Device:R_Small
Connections:
- net at C12.2, J6.4 (Pin_4), U13.3 (K)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: now also J6.3 (Pin_3)
- net at C11.2, J6.1 (Pin_1), U13.1 (K)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: now also J6.2 (Pin_2)
