File: INV_Board.kicad_pcb (KiCad board)
At the start: 4 copper layers, 84 x 66.5 mm, 194 parts, among them J3 Conn_01x06_Male, J4 Conn_01x06_Female, J5 Conn_01x08_Female, J6 Conn_01x08_Female, J7 Conn_01x05_Male, J8 Conn_01x02_Male, Q1 2N7002, Q2 AO3401A, Q3 CRSS037N10N, Q4 CRSS037N10N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

Commit message: Save progress
Parts:
- removed C49: CP_470uF+, Capacitor_THT:CP_Radial_D16.0mm_P7.50mm
- removed C63, C65, C66: C_0.1uF_100V, Capacitor_SMD:C_0603_1608Metric
- removed the D15 at (118.5, 96.5)
- removed the D17 at (145.0, 95.0)
- removed D18: D_TVS, Diode_SMD:D_0603_1608Metric
- removed R59, R61, R63: R_4k7, Resistor_SMD:R_0603_1608Metric
- removed R60, R62, R64: R_150, Resistor_SMD:R_0603_1608Metric
- removed TP1, TP2, TP3: TestPoint, TestPoint:TestPoint_Pad_D1.5mm
- added U12: SMF05CT1G, Package_TO_SOT_SMD:SOT-363_SC-70-6, F.Cu at (190.8, 104.6)
- added U13: SMF05CT1G, Package_TO_SOT_SMD:SOT-363_SC-70-6, F.Cu at (172.2, 127.8)
- added U14: SMF05CT1G, Package_TO_SOT_SMD:SOT-363_SC-70-6, F.Cu at (151.6, 124.5)
- J4, J5, J7: moved to F.Cu
- R1: footprint Resistor_SMD:R_0805_2012Metric -> Resistor_SMD:R_0603_1608Metric
- X1: footprint Oscillator:Oscillator_SMD_Abracon_ASE-4Pin_3.2x2.5mm -> INV_Board:X1OSC
- moved J6 152.7 mm to (196.2, 132.7), turned to 90 degrees
- moved C14 141.7 mm to (191.3, 132.1), turned to 180 degrees
- moved C15 140.8 mm to (191.3, 129.8), turned to 180 degrees
- moved R9 138.0 mm to (191.3, 126.7), turned to 180 degrees
- moved R8 137.2 mm to (187.5, 133.3), turned to 0 degrees
- moved C11 133.5 mm to (187.4, 131.3), turned to 180 degrees
- moved C12 132.6 mm to (187.4, 129.3), turned to 180 degrees
- moved C5 123.5 mm to (187.5, 127.3), turned to 0 degrees
- moved R1 121.6 mm to (191.8, 122.7)
- moved Q1 121.5 mm to (182.2, 122.7)
- moved Q2 120.7 mm to (187.3, 123.1)
- moved U2 116.8 mm to (179.6, 128.5), turned to 180 degrees
- moved J4 110.9 mm to (197.4, 103.5), turned to -90 degrees
- moved C21 99.8 mm to (118.9, 114.8)
- moved U5 97.3 mm to (123.4, 114.8)
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Connections:
- J5 pad 7: I2CSDA -> I2CSCL
- R20 pad 2: Net-(J7-Pad3) -> Net-(J7-Pad2)
- R21 pad 2: I2CSDA -> I2CSCL
- R27 pad 2: Net-(J7-Pad2) -> Net-(J7-Pad3)
- U1 pad 11: ISU_MCU -> unconnected-(U1-Pad11)
- U1 pad 17: ISV_MCU -> unconnected-(U1-Pad17)
- U1 pad 18: ISW_MCU -> unconnected-(U1-Pad18)
- U1 pad 46: I2CSDA -> I2CSCL
- U5 pad 9: (no net) -> SGU
- U8 pad 9: (no net) -> SGU
- X1 pad 2: GND -> SGU
- X1 pad 3: Net-(U2-Pad5) -> Net-(U1-Pad5)
Routing:
- net +12V: track 0.65 -> 176.1 mm, vias 0 -> 6
- net SGU: track 0.00 -> 36.3 mm, vias 104 -> 108
- net ISW: track 0.00 -> 28.9 mm, vias 0 -> 2
- net /VGH: track 0.00 -> 24.1 mm
- net Net-(R45-Pad1): track 0.00 -> 23.4 mm, vias 0 -> 2
- net /VGL: track 0.00 -> 22.2 mm, vias 1 -> 2
- net /WGL: track 0.00 -> 20.0 mm, vias 0 -> 2
- net +VDC: track 10.5 -> 24.2 mm, vias 177 -> 194
- net Net-(C8-Pad1): track 0.00 -> 12.0 mm, vias 0 -> 2
- net SWW: track 0.00 -> 11.9 mm
- net PhaseW: track 0.00 -> 11.9 mm
- net Net-(R3-Pad2): track 0.00 -> 9.21 mm
- net SWV: track 0.00 -> 7.48 mm
- net /WGH: track 0.00 -> 7.29 mm
- net Net-(C38-Pad1): track 0.00 -> 6.32 mm
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- added copper zone on F.Cu, net +12V
- added copper zone on F.Cu, net Net-(C8-Pad2)
Other:
- board size 84 x 66.5 mm -> 84.1 x 87.1 mm
- board text removed: "#Res N/C SWO SWC SWDIO G"
- board text removed: "3v3"
- board text removed: "5V 3V3 G An Rx Tx An An"
- board text removed: "G 5V PWM"
- board text removed: "G H3 H2 H1 N/C 5V"
- board text removed: "I_PhU TP"
- board text removed: "I_PhV TP"
- board text removed: "I_PhW TP"
- board text removed: "PhU"
- board text removed: "PhV"
- board text removed: "PhW"
- board text removed: "SDA SCL 3v3 G"
- board text removed: "USB B Micro"

Commit message: Update progress
Parts:
- removed C14, C15: C_4.7nF, Capacitor_SMD:C_0603_1608Metric
- removed R8, R9: R_60, Resistor_SMD:R_0603_1608Metric
- added G***: LOGO, LOGO, B.Cu at (129.4, 58.2)
- added G***: LOGO, LOGO, B.Cu at (157.1, 78.5)
- C41, C42, C46, J8: moved to F.Cu
- moved U12 14.1 mm to (177.9, 110.6)
- moved J4 10.0 mm to (196.2, 113.4), turned to 90 degrees
- moved D22 8.24 mm to (176.0, 84.2), turned to 180 degrees
- moved C71 7.92 mm to (155.4, 105.0)
- moved U13 7.37 mm to (177.7, 132.7)
- moved R66 4.79 mm to (157.5, 107.2)
- moved R5 4.55 mm to (182.2, 108.0)
- moved R10 4.47 mm to (182.2, 110.0)
- moved R12 4.36 mm to (182.2, 112.0)
- moved R65 3.94 mm to (163.3, 103.5)
- moved D19 2.42 mm to (157.2, 113.2)
- moved C16 2.19 mm to (191.8, 113.0)
- moved C20 2.19 mm to (186.7, 113.0)
- moved R15 2.19 mm to (186.7, 109.2)
- moved R7 2.19 mm to (191.8, 109.2)
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Connections:
- J5 pad 7: I2CSCL -> I2CSDA
- J6 pad 2: Net-(C14-Pad1) -> Net-(C11-Pad2)
- J6 pad 3: Net-(C15-Pad1) -> Net-(C12-Pad2)
- R21 pad 2: I2CSCL -> I2CSDA
- U1 pad 46: I2CSCL -> I2CSDA
- U12 pad 3: Net-(J4-Pad2) -> Motor_T
- U12 pad 6: Motor_T -> Net-(J4-Pad2)
- U14 pad 3: I2CSCL -> I2CSDA
Routing:
- net +3V3: track 2.37 -> 260.9 mm, vias 0 -> 13
- net +5V: track 0.00 -> 134.7 mm
- net SWDIO: track 0.00 -> 67.7 mm, vias 0 -> 1
- net SGU: track 36.3 -> 102.8 mm, vias 108 -> 280
- net BoardTemp: track 0.00 -> 65.1 mm, vias 0 -> 3
- net SWCLK: track 0.00 -> 59.2 mm, vias 0 -> 1
- net #RES: track 0.00 -> 56.5 mm, vias 0 -> 1
- net SWO: track 0.00 -> 55.9 mm, vias 0 -> 1
- net WHin: track 2.77 -> 57.8 mm, vias 1 -> 2
- net WLin: track 3.02 -> 54.7 mm, vias 1 -> 2
- net +12V: track 176.1 -> 222.0 mm, vias 6 -> 7
- net AnalogIn: track 0.00 -> 41.6 mm, vias 0 -> 2
- net I2CSDA: track 0.00 -> 40.6 mm, vias 0 -> 2
- net PhaseW: track 11.9 -> 51.3 mm, vias 0 -> 2
- net I2CSCL: track 0.00 -> 39.1 mm, vias 0 -> 1
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- added copper zone on F.Cu, net +3V3
- added copper zone on F.Cu, net +5V
- added copper zone on F.Cu, net Net-(C25-Pad2)
- added copper zone on F.Cu, net Net-(C37-Pad2)
- added copper zone on B.Cu, net SGU
- added copper zone on In1.Cu, net SGU
- added copper zone on In2.Cu, net SGU
- added copper zone on In2.Cu, net SWU
- added copper zone on In2.Cu, net SWV
- added copper zone on In2.Cu, net SWW
Other:
- outline, holes or cut-outs redrawn
- board text added: "+12VBuck"
- board text added: "ANA_IO"
- board text added: "CAN_BUS"
- board text added: "DEBUG"
- board text added: "Digi_IO"
- board text added: "G"
- board text added: "HALL_SEN"
- board text added: "HEARTBEAT"
- board text added: "MTR_V"
- board text added: "MTR_W"
- board text added: "P+"
- board text added: "P3V3"
- board text added: "P5V"
- board text removed: "5v0"
